File: toaster-reflow.kicad_pcb (KiCad board)
At the start: 2 copper layers, 0 parts

Commit message: Forgot a footprint! Created components on board
Parts:
- added C1: 0.1uF, Capacitor_SMD:C_0603_1608Metric, F.Cu at (85.0, 87.1)
- added C10: 0.1uF, Capacitor_SMD:C_0603_1608Metric, F.Cu at (187.3, 76.0)
- added C11: 0.1uF, Capacitor_SMD:C_0603_1608Metric, F.Cu at (184.3, 75.6)
- added C2: 0.01uF, Capacitor_SMD:C_0603_1608Metric, F.Cu at (78.2, 135.0)
- added C3: 0.1uF, Capacitor_SMD:C_0603_1608Metric, F.Cu at (81.2, 135.0)
- added C4: 0.01uF, Capacitor_SMD:C_0603_1608Metric, F.Cu at (84.2, 135.3)
- added C5: 0.1uF, Capacitor_SMD:C_0603_1608Metric, F.Cu at (89.2, 131.8)
- added C6: 0.1uF, Capacitor_SMD:C_0603_1608Metric, F.Cu at (87.2, 135.3)
- added C7: 0.01uF, Capacitor_SMD:C_0603_1608Metric, F.Cu at (192.3, 74.0)
- added C8: 0.1uF, Capacitor_SMD:C_0603_1608Metric, F.Cu at (190.3, 76.0)
- added C9: 0.01uF, Capacitor_SMD:C_0603_1608Metric, F.Cu at (192.3, 72.4)
- added D1: 400V 1A, Diode_SMD:D_SMA, F.Cu at (77.2, 119.7)
- added D2: RED, Diode_SMD:D_0603_1608Metric, F.Cu at (124.8, 75.7)
- added D3: GREEN, Diode_SMD:D_0603_1608Metric, F.Cu at (88.5, 83.6)
- added D4: RED, Diode_SMD:D_0603_1608Metric, F.Cu at (75.2, 135.0)
- added D5: RED, Diode_SMD:D_0603_1608Metric, F.Cu at (178.3, 75.7)
- added J1: 1935161, 1935161:PHOENIX_1935161, F.Cu at (128.6, 70.3)
- added J2: 1935161, 1935161:PHOENIX_1935161, F.Cu at (115.7, 83.2)
- added J3: Raspberry_Pi_2_3, Connector_PinHeader_2.54mm:PinHeader_2x20_P2.54mm_Vertical, F.Cu at (75.5, 67.9)
- added J4: 1935161, 1935161:PHOENIX_1935161, F.Cu at (78.9, 129.6)
- added J5: 1935161, 1935161:PHOENIX_1935161, F.Cu at (182.0, 70.3)
- added J6: Conn_01x03, Connector_PinSocket_2.54mm:PinSocket_1x03_P2.54mm_Vertical, F.Cu at (81.7, 81.1)
- added K1: 1-1415899-3, 1-1415899-3:RELAY_1-1415899-3, F.Cu at (95.7, 72.7)
- added LS1: Speaker, PS12:PS12, F.Cu at (116.9, 72.5)
- added Q1: Q_PMOS_GSD, Package_TO_SOT_SMD:SOT-23, F.Cu at (85.2, 84.6)
- added Q2: Q_PMOS_GSD, Package_TO_SOT_SMD:SOT-23, F.Cu at (88.6, 81.1)
- added Q3: Q_PMOS_GSD, Package_TO_SOT_SMD:SOT-23, F.Cu at (81.6, 89.8)
- added Q4: Q_PMOS_GSD, Package_TO_SOT_SMD:SOT-23, F.Cu at (85.9, 132.8)
- added Q5: Q_PMOS_GSD, Package_TO_SOT_SMD:SOT-23, F.Cu at (189.0, 73.5)
- added R1: 10K, Resistor_SMD:R_0603_1608Metric, F.Cu at (81.4, 92.3)
- added R2: 470, Resistor_SMD:R_0603_1608Metric, F.Cu at (88.4, 85.2)
- added R3: 260, Resistor_SMD:R_0603_1608Metric, F.Cu at (91.4, 85.2)
- added R4: 10K, Resistor_SMD:R_0603_1608Metric, F.Cu at (91.9, 81.6)
- added R5: 1K, Resistor_SMD:R_0603_1608Metric, F.Cu at (84.8, 88.7)
- added R6: 10K, Resistor_SMD:R_0603_1608Metric, F.Cu at (91.9, 80.0)
- added R7: 470, Resistor_SMD:R_0603_1608Metric, F.Cu at (89.2, 133.3)
- added R8: 470, Resistor_SMD:R_0603_1608Metric, F.Cu at (181.3, 75.6)
- added U1: 3.3V Ref, Package_TO_SOT_SMD:SOT-23, F.Cu at (85.2, 81.1)
- added U2: MAX31856, Package_SO:TSSOP-14_4.4x5mm_P0.65mm, F.Cu at (88.2, 128.2)
- added U3: MAX31856, Package_SO:TSSOP-14_4.4x5mm_P0.65mm, F.Cu at (191.3, 68.9)

Commit message: Finish pcb routing
Parts:
- moved J3 94.1 mm to (163.8, 100.3)
- moved D4 83.2 mm to (157.5, 147.3), turned to 90 degrees
- moved C7 83.0 mm to (138.4, 137.2), turned to 90 degrees
- moved J5 80.4 mm to (132.1, 133.3), turned to 270 degrees
- moved U3 80.2 mm to (143.5, 133.3)
- moved Q2 79.0 mm to (159.0, 116.8), turned to 180 degrees
- moved R5 78.6 mm to (160.0, 111.8), turned to 90 degrees
- moved C9 78.5 mm to (138.4, 129.5), turned to 90 degrees
- moved C8 77.4 mm to (138.4, 133.3), turned to 90 degrees
- moved C10 76.0 mm to (142.2, 137.2)
- moved Q1 74.6 mm to (153.7, 114.3)
- moved R1 74.6 mm to (153.7, 110.5), turned to 180 degrees
- moved U1 74.2 mm to (143.5, 127.0)
- moved J6 74.0 mm to (154.9, 91.4)
- moved Q3 73.1 mm to (153.7, 101.6), turned to 270 degrees
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Routing:
- net +3V3: track 0.00 -> 110.2 mm, vias 0 -> 4
- net +5V: track 0.00 -> 73.1 mm, vias 0 -> 1
- net /THERMO1_DRDY: track 0.00 -> 48.0 mm, vias 0 -> 1
- net /HEAT_ENABLE: track 0.00 -> 46.3 mm, vias 0 -> 1
- net /THERMO1_CS: track 0.00 -> 45.3 mm
- net /THERMO1_FAULT: track 0.00 -> 44.7 mm, vias 0 -> 3
- net /BUZZER: track 0.00 -> 43.5 mm, vias 0 -> 2
- net /THERMO2_DRDY: track 0.00 -> 43.3 mm, vias 0 -> 3
- net /THERMO_SCK: track 0.00 -> 36.0 mm, vias 0 -> 2
- net /THERMO_MOSI: track 0.00 -> 35.9 mm, vias 0 -> 2
- net /THERMO_MISO: track 0.00 -> 34.9 mm
- net /THERMO2_FAULT: track 0.00 -> 30.8 mm, vias 0 -> 3
- net Net-(D1-Pad1): track 0.00 -> 30.7 mm, vias 0 -> 2
- net +3.3VADC: track 0.00 -> 24.8 mm
- net Net-(C8-Pad2): track 0.00 -> 23.5 mm, vias 0 -> 1
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- added copper zone on B.Cu, net GND
- added copper zone on F.Cu, net GND
Other:
- board outline added: 41.9 x 63.5 mm
- net class 3A added: clearance 0.2, trace_width 1.37, via_dia 0.8, via_drill 0.4
- net class AC_Load added: clearance 0.2, trace_width 3, via_dia 0.8, via_drill 0.4
- net class THERMOCOUPLE added: clearance 0.25, trace_width 0.25, via_dia 0.8, via_drill 0.4
- board text added: "- 5V +"
- board text added: "Heating"
- board text added: "Power"
- board text added: "Servo"
