File: toaster-reflow.kicad_pcb (KiCad board)
At the start: 2 copper layers, 56 x 65 mm, 47 parts, among them J1 1935161, J2 1935161, J3 Raspberry_Pi_2_3, J4 Conn_01x04, J6 Conn_01x03, K1 1-1415899-3, Q1 Q_NMOS_GSD, Q2 Q_NMOS_GSD, Q3 Q_PNP_BEC, Q4 Q_PNP_BEC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

Commit message: send out for fabrication
Other:
- board text added: "+"
- board text added: "+- T2"
- board text added: "-"
- board text added: "Joe Hirschfeld"
- board text added: "PWR"
- board text added: "Rev 1"
- board text added: "Switch 250VAC 12A"
- board text added: "T1 +-"
- board text added: "ToasterBoard"
- board text removed: "Switch 250VAC@12A"
